File: eca/eca.kicad_sch (KiCad schematic)
At the start: 22 parts, among them J1 RPI Bus, J10 ESP32CAM Power Supply Bus, J11 28BYJ48 1 Power Supply Bus, J12 28BYJ48 2 Power Supply Bus, J13 28BYJ48 3 Power Supply Bus, J14 Power Supply Input, J2 GY 906 Bus, J3 MAX30102 Bus, J4 TCRT5000 1 Bus, J5 TCRT5000 2 Bus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

Commit message: added fan bus
Parts:
- removed C5: 100nF, Capacitor_THT:C_Disc_D4.3mm_W1.9mm_P5.00mm, symbol Device:C
- removed J6: TCRT5000 3 Bus, Connector_PinHeader_2.54mm:PinHeader_1x04_P2.54mm_Vertical, symbol Connector:Conn_01x04_Pin
- added J15: Fan 1 Power Supply Bus, Connector_PinHeader_2.54mm:PinHeader_1x02_P2.54mm_Vertical, symbol Connector:Conn_01x02_Pin
- added J16: Fan Power Supply Bus, Connector_PinHeader_2.54mm:PinHeader_1x02_P2.54mm_Vertical, symbol Connector:Conn_01x02_Pin
- C1: footprint CP_Radial_D4.0mm_P1.50mm -> Capacitor_THT:CP_Radial_D8.0mm_P5.00mm
Connections:
- net 5V: now also J15.1 (Pin_1), J16.1 (Pin_1)
- net GND: now also J15.2 (Pin_2), J16.2 (Pin_2)
Other:
- moved on the sheet: C2, J10, J8

Commit message: changed input connector
Parts:
- J14: footprint Connector_PinHeader_2.54mm:PinHeader_1x02_P2.54mm_Vertical -> TerminalBlock:TerminalBlock_Xinya_XY308-2.54-2P_1x02_P2.54mm_Horizontal
Changed lines of the file:
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@@
 			)
 		)
-		(property "Footprint" "Connector_PinHeader_2.54mm:PinHeader_1x02_P2.54mm_Vertical"
+		(property "Footprint" "TerminalBlock:TerminalBlock_Xinya_XY308-2.54-2P_1x02_P2.54mm_Horizontal"
 			(at 209.55 113.03 0)
 			(effects

Commit message: alpha version
Parts:
- removed C3, C4: 100nF, Capacitor_THT:C_Disc_D4.3mm_W1.9mm_P5.00mm, symbol Device:C
- removed J14: Power Supply Input, TerminalBlock:TerminalBlock_Xinya_XY308-2.54-2P_1x02_P2.54mm_Horizontal, symbol Connector:Conn_01x02_Pin
- added J6: Power Supply Input, TerminalBlock:TerminalBlock_Xinya_XY308-2.54-3P_1x03_P2.54mm_Horizontal, symbol Connector:Conn_01x03_Pin
Connections:
- net 3.3V: now also J1.18 (Pin_18), J1.2 (Pin_2); no longer J1.1 (Pin_1), J1.17 (Pin_17)
- net 5V: now also J1.1 (Pin_1), J1.3 (Pin_3), J6.1 (Pin_1); no longer J1.2 (Pin_2), J1.4 (Pin_4)
- net GND: now also J1.10 (Pin_10), J1.13 (Pin_13), J1.19 (Pin_19), J1.26 (Pin_26), J1.29 (Pin_29), J1.33 (Pin_33), J1.40 (Pin_40), J1.5 (Pin_5), J6.3 (Pin_3); no longer J1.14 (Pin_14), J1.20 (Pin_20), J1.25 (Pin_25), J1.30 (Pin_30), J1.34 (Pin_34), J1.39 (Pin_39), J1.6 (Pin_6), J1.9 (Pin_9)
- net GPIO10: now also J1.20 (Pin_20); no longer J1.19 (Pin_19)
- net GPIO11: now also J1.24 (Pin_24); no longer J1.23 (Pin_23)
- net GPIO12: now also J1.31 (Pin_31); no longer J1.32 (Pin_32)
- net GPIO13: now also J1.34 (Pin_34); no longer J1.33 (Pin_33)
- net GPIO14: now also J1.7 (Pin_7); no longer J1.8 (Pin_8)
- net GPIO15: now also J1.9 (Pin_9); no longer J1.10 (Pin_10)
- net GPIO16: now also J1.35 (Pin_35); no longer J1.36 (Pin_36)
- net GPIO17: now also J1.12 (Pin_12); no longer J1.11 (Pin_11)
- net GPIO18: now also J1.11 (Pin_11); no longer J1.12 (Pin_12)
- net GPIO19: now also J1.36 (Pin_36); no longer J1.35 (Pin_35)
- net GPIO2: now also J1.4 (Pin_4); no longer J1.3 (Pin_3)
- net GPIO20: now also J1.37 (Pin_37); no longer J1.38 (Pin_38)
- net GPIO21: now also J1.39 (Pin_39); no longer J1.40 (Pin_40)
- net GPIO22: now also J1.16 (Pin_16); no longer J1.15 (Pin_15)
- net GPIO23: now also J1.15 (Pin_15); no longer J1.16 (Pin_16)
- net GPIO24: now also J1.17 (Pin_17); no longer J1.18 (Pin_18)
- net GPIO25: now also J1.21 (Pin_21); no longer J1.22 (Pin_22)
- net GPIO26: now also J1.38 (Pin_38); no longer J1.37 (Pin_37)
- net GPIO27: now also J1.14 (Pin_14); no longer J1.13 (Pin_13)
- net GPIO3: now also J1.6 (Pin_6); no longer J1.5 (Pin_5)
- net GPIO4: now also J1.8 (Pin_8); no longer J1.7 (Pin_7)
- net GPIO5: now also J1.30 (Pin_30); no longer J1.29 (Pin_29)
- net GPIO6: now also J1.32 (Pin_32); no longer J1.31 (Pin_31)
- net GPIO7: now also J1.25 (Pin_25); no longer J1.26 (Pin_26)
- net GPIO8: now also J1.23 (Pin_23); no longer J1.24 (Pin_24)
- net GPIO9: now also J1.22 (Pin_22); no longer J1.21 (Pin_21)
- net ID_SC: now also J1.27 (Pin_27); no longer J1.28 (Pin_28)
- net ID_SD: now also J1.28 (Pin_28); no longer J1.27 (Pin_27)
Other:
- moved on the sheet: C6, C7, C8, J2, J3, J4, J5
